Commit message: Added camera and lidar to URDF models and tested with Gazebo

File: arm_description/urdf/arm.gazebo.xacro (robot description, xacro)
@@ -1,18 +1,52 @@
 <?xml version="1.0"?>
 <robot xmlns:xacro="http://ros.org/wiki/xacro">
-    <xacro:macro name="arm_gazebo">
-        <xacro:macro name="arm_link" params="link">
-            <gazebo reference="arm_link_${link}">
-                <material>Gazebo/Blue</material>
-                <mu1>0.2</mu1>
-                <mu2>0.2</mu2>
-            </gazebo>
-        </xacro:macro>
-        <xacro:arm_link link="1"/>
-        <xacro:arm_link link="2"/>
-        <xacro:arm_link link="3"/>
-        <xacro:arm_link link="4"/>
-        <xacro:arm_link link="5"/>
-        <xacro:arm_link link="6"/>
+    <xacro:macro name="arm_link" params="link">
+        <gazebo reference="arm_link_${link}">
+            <material>Gazebo/Blue</material>
+            <mu1>0.2</mu1>
+            <mu2>0.2</mu2>
+        </gazebo>
     </xacro:macro>
+    <xacro:arm_link link="1"/>
+    <xacro:arm_link link="2"/>
+    <xacro:arm_link link="3"/>
+    <xacro:arm_link link="4"/>
+    <xacro:arm_link link="5"/>
+    <xacro:arm_link link="6"/>
+    <gazebo reference="arm_camera_link">
+        <sensor type="camera" name="camera">
+            <update_rate>30.0</update_rate>
+            <camera name="front">
+                <horizontal_fov>1.3962634</horizontal_fov>
+                <image>
+                    <width>800</width>
+                    <height>600</height>
+                    <format>R8G8B8</format>
+                </image>
+                <clip>
+                    <near>0.02</near>
+                    <far>300</far>
+                </clip>
+                <noise>
+                    <type>gaussian</type>
+                    <mean>0.0</mean>
+                    <stddev>0.007</stddev>
+                </noise>
+            </camera>
+            <plugin name="camera_controller" filename="libgazebo_ros_camera.so">
+                <alwaysOn>true</alwaysOn>
+                <updateRate>0.0</updateRate>
+                <cameraName>arm_camera</cameraName>
+                <imageTopicName>image_raw</imageTopicName>
+                <cameraInfoTopicName>camera_info</cameraInfoTopicName>
+                <frameName>arm_camera_link</frameName>
+                <hackBaseline>0.07</hackBaseline>
+                <distortionK1>0.0</distortionK1>
+                <distortionK2>0.0</distortionK2>
+                <distortionK3>0.0</distortionK3>
+                <distortionT1>0.0</distortionT1>
+                <distortionT2>0.0</distortionT2>
+            </plugin>
+        </sensor>
+    </gazebo>
 </robot>

File: arm_description/urdf/arm.urdf.xacro (robot description, xacro)
@@ -185,4 +185,31 @@
             </collision>
         </link>
+        <joint name="arm_camera_attachment" type="fixed">
+            <parent link="arm_link_6"/>
+            <child link="arm_camera_link"/>
+            <origin xyz="0.09 -0.025 0.065" rpy="0.0 0.0 0.0"/>
+        </joint>
+        <link name="arm_camera_link">
+            <inertial>
+                <origin xyz="0.0 0.0 0.0" rpy="0.0 0.0 0.0"/>
+                <mass value="0.1"/>
+                <inertia ixx="0.001" ixy="0.0" ixz="0.0" iyy="0.001" iyz="0.0" izz="0.001"/>
+            </inertial>
+            <visual>
+                <origin xyz="0.0 0.0 0.0" rpy="0.0 0.0 0.0"/>
+                <geometry>
+                    <mesh filename="package://arm_description/meshes/visual/arm_camera.stl" scale="0.001 0.001 0.001"/>
+                </geometry>
+                <material name="Grey">
+                    <color rgba="0.2 0.2 0.2 1"/>
+                </material>
+            </visual>
+            <collision>
+                <origin xyz="0.0 0.0 0.0" rpy="0.0 0.0 0.0"/>
+                <geometry>
+                    <mesh filename="package://arm_description/meshes/collision/arm_camera.stl" scale="0.001 0.001 0.001"/>
+                </geometry>
+            </collision>
+        </link>
         <xacro:include filename="$(find arm_description)/urdf/arm.transmission.xacro"/>
     </xacro:macro>

File: arm_description/urdf/arm.xacro (robot description, xacro)
@@ -11,5 +11,9 @@
         <origin xyz="0 0 0" rpy="0 0 0"/>
     </joint>
-    <xacro:include filename="$(find arm_description)/urdf/common.gazebo.xacro"/>
-    <xacro:include filename="$(find arm_description)/urdf/arm.transmission.xacro"/>
+    <xacro:include filename="$(find arm_description)/urdf/arm.gazebo.xacro"/>
+    <gazebo>
+        <plugin name="ros_control" filename="libgazebo_ros_control.so">
+          <robotNamespace></robotNamespace>
+        </plugin>
+    </gazebo>
 </robot>

File: hexapod_description/urdf/hexapod.gazebo.xacro (robot description, xacro)
@@ -1,6 +1,104 @@
 <?xml version="1.0"?>
 <robot xmlns:xacro="http://ros.org/wiki/xacro">
-    <xacro:macro name="hexapod_gazebo">
-        <gazebo reference="body_link">
+    <gazebo reference="body_link">
+        <material>Gazebo/Black</material>
+        <mu1>0.2</mu1>
+        <mu2>0.2</mu2>
+        <maxVel>0</maxVel>
+    </gazebo>
+    <gazebo reference="front_camera_link">
+        <sensor type="camera" name="camera">
+            <update_rate>30.0</update_rate>
+            <camera name="front">
+                <horizontal_fov>1.3962634</horizontal_fov>
+                <image>
+                    <width>800</width>
+                    <height>600</height>
+                    <format>R8G8B8</format>
+                </image>
+                <clip>
+                    <near>0.02</near>
+                    <far>300</far>
+                </clip>
+                <noise>
+                    <type>gaussian</type>
+                    <mean>0.0</mean>
+                    <stddev>0.007</stddev>
+                </noise>
+            </camera>
+            <plugin name="camera_controller" filename="libgazebo_ros_camera.so">
+                <alwaysOn>true</alwaysOn>
+                <updateRate>0.0</updateRate>
+                <cameraName>front_camera</cameraName>
+                <imageTopicName>image_raw</imageTopicName>
+                <cameraInfoTopicName>camera_info</cameraInfoTopicName>
+                <frameName>front_camera_link</frameName>
+                <hackBaseline>0.07</hackBaseline>
+                <distortionK1>0.0</distortionK1>
+                <distortionK2>0.0</distortionK2>
+                <distortionK3>0.0</distortionK3>
+                <distortionT1>0.0</distortionT1>
+                <distortionT2>0.0</distortionT2>
+            </plugin>
+        </sensor>
+    </gazebo>
+    <gazebo reference="lidar_link">
+        <sensor type="ray" name="lidar">
+            <pose>0 0 0 0 0 0</pose>
+            <visualize>false</visualize>
+            <update_rate>20</update_rate>
+            <ray>
+                <scan>
+                    <horizontal>
+                        <samples>102</samples>
+                        <resolution>1</resolution>
+                        <min_angle>-0.8901</min_angle>
+                        <max_angle>0.8901</max_angle>
+                    </horizontal>
+                    <vertical>
+                        <samples>9</samples>
+                        <resolution>1</resolution>
+                        <min_angle>-0.0785</min_angle>
+                        <max_angle>0.0785</max_angle>
+                    </vertical>
+                </scan>
+                <range>
+                    <min>0.2</min>
+                    <max>4</max>
+                    <resolution>0.01</resolution>
+                </range>
+                <noise>
+                    <type>gaussian</type>
+                    <mean>0.0</mean>
+                    <stddev>0.0</stddev>
+                </noise>
+            </ray>
+            <plugin name="gazebo_ros_head_lidar_controller" filename="libgazebo_ros_laser.so">
+                <robotNamespace></robotNamespace>
+                <topicName>laser_scan</topicName>
+                <frameName>lidar_link</frameName>
+            </plugin>
+        </sensor>
+    </gazebo>
+    <xacro:leg_gazebo suffix="lf"/>
+    <xacro:leg_gazebo suffix="lm"/>
+    <xacro:leg_gazebo suffix="lr"/>
+    <xacro:leg_gazebo suffix="rf"/>
+    <xacro:leg_gazebo suffix="rm"/>
+    <xacro:leg_gazebo suffix="rr"/>
+    <xacro:macro name="leg_gazebo" params="suffix">
+        <gazebo reference="coxa_link_${suffix}">
+            <material>Gazebo/White</material>
+            <mu1>0.2</mu1>
+            <mu2>0.2</mu2>
+            <maxVel>0</maxVel>
+        </gazebo>
+        <gazebo reference="thigh_link_${suffix}">
+            <material>Gazebo/Grey</material>
+            <mu1>0.2</mu1>
+            <mu2>0.2</mu2>
+            <maxVel>0</maxVel>
+        </gazebo>
+        <gazebo reference="tibia_link_${suffix}">
             <material>Gazebo/Black</material>
             <mu1>0.2</mu1>
@@ -8,30 +106,4 @@
             <maxVel>0</maxVel>
         </gazebo>
-        <xacro:leg_gazebo suffix="lf"/>
-        <xacro:leg_gazebo suffix="lm"/>
-        <xacro:leg_gazebo suffix="lr"/>
-        <xacro:leg_gazebo suffix="rf"/>
-        <xacro:leg_gazebo suffix="rm"/>
-        <xacro:leg_gazebo suffix="rr"/>
     </xacro:macro>
-    <xacro:macro name="leg_gazebo" params="suffix">
-            <gazebo reference="coxa_link_${suffix}">
-                <material>Gazebo/White</material>
-                <mu1>0.2</mu1>
-                <mu2>0.2</mu2>
-                <maxVel>0</maxVel>
-            </gazebo>
-            <gazebo reference="thigh_link_${suffix}">
-                <material>Gazebo/Grey</material>
-                <mu1>0.2</mu1>
-                <mu2>0.2</mu2>
-                <maxVel>0</maxVel>
-            </gazebo>
-            <gazebo reference="tibia_link_${suffix}">
-                <material>Gazebo/Black</material>
-                <mu1>0.2</mu1>
-                <mu2>0.2</mu2>
-                <maxVel>0</maxVel>
-            </gazebo>
-        </xacro:macro>
 </robot>

File: hexapod_description/urdf/hexapod.urdf.xacro (robot description, xacro)
@@ -35,4 +35,58 @@
         <xacro:hexapod_leg xyz="0.0 -0.0795 0.0" rpy="0.0 0.0 -${pi/2.0}" suffix="rm"/>
         <xacro:hexapod_leg xyz="-0.1497 -0.0797 0.0" rpy="0.0 0.0 -2.404" suffix="rr"/>
+        <joint name="camera_attachment" type="fixed">
+            <parent link="body_link"/>
+            <child link="front_camera_link"/>
+            <origin xyz="0.33 0.0 0.04" rpy="0.0 0.0 0.0"/>
+        </joint>
+        <link name="front_camera_link">
+            <inertial>
+                <origin xyz="0.0 0.0 0.0" rpy="0.0 0.0 0.0"/>
+                <mass value="1"/>
+                <inertia ixx="0.001" ixy="0.0" ixz="0.0" iyy="0.001" iyz="0.0" izz="0.001"/>
+            </inertial>
+            <visual>
+                <origin xyz="0 0 0.0" rpy="0.0 0.0 0.0"/>
+                <geometry>
+                    <mesh filename="package://hexapod_description/meshes/visual/camera.stl" scale="0.001 0.001 0.001"/>
+                </geometry>
+                <material name="Grey">
+                    <color rgba="0.2 0.2 0.2 1"/>
+                </material>
+            </visual>
+            <collision>
+                <origin xyz="0.0 0.0 0.0" rpy="0.0 0.0 0.0"/>
+                <geometry>
+                    <mesh filename="package://hexapod_description/meshes/collision/camera.stl" scale="0.001 0.001 0.001"/>
+                </geometry>
+            </collision>
+        </link>
+        <joint name="lidar_attachment" type="fixed">
+            <parent link="body_link"/>
+            <child link="lidar_link"/>
+            <origin xyz="0.275 0.0 0.079" rpy="0.0 0.0 0.0"/>
+        </joint>
+        <link name="lidar_link">
+            <inertial>
+                <origin xyz="0.0 0.0 0.0" rpy="0.0 0.0 0.0"/>
+                <mass value="1"/>
+                <inertia ixx="0.001" ixy="0.0" ixz="0.0" iyy="0.001" iyz="0.0" izz="0.001"/>
+            </inertial>
+            <visual>
+                <origin xyz="0.0 0.0 0.0" rpy="0.0 0.0 0.0"/>
+                <geometry>
+                    <mesh filename="package://hexapod_description/meshes/visual/lidar.stl" scale="0.001 0.001 0.001"/>
+                </geometry>
+                <material name="Grey">
+                    <color rgba="0.2 0.2 0.2 1"/>
+                </material>
+            </visual>
+            <collision>
+                <origin xyz="0.0 0.0 0.0" rpy="0.0 0.0 0.0"/>
+                <geometry>
+                    <mesh filename="package://hexapod_description/meshes/collision/lidar.stl" scale="0.001 0.001 0.001"/>
+                </geometry>
+            </collision>
+        </link>
     </xacro:macro>
     <xacro:macro name="hexapod_leg" params="xyz rpy suffix">

File: hexapod_description/urdf/hexapod_arm.xacro (robot description, xacro)
@@ -8,7 +8,5 @@
     <!--Include Gazebo components-->
     <xacro:include filename="$(find hexapod_description)/urdf/hexapod.gazebo.xacro"/>
-    <xacro:hexapod_gazebo/>
     <xacro:include filename="$(find arm_description)/urdf/arm.gazebo.xacro"/>
-    <xacro:arm_gazebo/>
     <gazebo>
         <plugin name="ros_control" filename="libgazebo_ros_control.so">
