Commit message: Completed hexapod URDF model, combined both into a single model

File: arm_description/urdf/arm.urdf.xacro (robot description, xacro)
@@ -1,186 +1,188 @@
 <?xml version="1.0" ?>
 <robot xmlns:xacro="http://www.ros.org/wiki/xacro">
-<xacro:macro name="hexapod_arm" params="parent">
-    <joint name="arm_attachment" type="fixed">
-        <parent link="${parent}"/>
-        <child link="arm_link_1"/>
-    </joint>
-    <link name="arm_link_1">
-        <inertial>
-            <origin xyz="0.0 0.0 0.0" rpy="0.0 0.0 0.0"/>
-            <mass value="0.1"/>
-            <inertia ixx="0.001" ixy="0.001" ixz="0.001" iyy="0.001" iyz="0.001" izz="0.001"/>
-        </inertial>
-        <visual>
-            <origin xyz="0 0 0.0" rpy="0.0 0.0 0.0"/>
-            <geometry>
-                <mesh filename="package://arm_description/meshes/visual/arm_link_1.stl" scale="0.001 0.001 0.001"/>
-            </geometry>
-            <material name="Grey">
-                <color rgba="0.2 0.2 0.2 1"/>
-            </material>
-        </visual>
-        <collision>
-            <origin xyz="0.0 0.0 0.0" rpy="0.0 0.0 0.0"/>
-            <geometry>
-                <mesh filename="package://arm_description/meshes/collision/arm_link_1.stl" scale="0.001 0.001 0.001"/>
-            </geometry>
-        </collision>
-    </link>
-    <joint name="arm_joint_1" type="revolute">
-        <parent link="arm_link_1"/>
-        <child link="arm_link_2"/>
-        <origin xyz="0.0 0.0 0.194" rpy="0.0 0.0 0.0"/>
-        <axis xyz="0 0 1"/>
-        <dynamics damping="0"/>
-        <dynamics friction="0"/>
-        <limit effort="87" velocity="5.6548668" lower="-2.6179939" upper="2.6179939" />
-    </joint>
-    <link name="arm_link_2">
-        <inertial>
-            <origin xyz="0.0 0.0 0.0" rpy="0.0 0.0 0.0"/>
-            <mass value="0.1"/>
-            <inertia ixx="0.001" ixy="0.001" ixz="0.001" iyy="0.001" iyz="0.001" izz="0.001"/>
-        </inertial>
-        <visual>
-            <origin xyz="0.0 0.0 0.0" rpy="0.0 0.0 0.0"/>
-            <geometry>
-                <mesh filename="package://arm_description/meshes/visual/arm_link_2.stl" scale="0.001 0.001 0.001"/>
-            </geometry>
-            <material name="Grey">
-                <color rgba="0.2 0.2 0.2 1"/>
-            </material>
-        </visual>
-        <collision>
-            <origin xyz="0.0 0.0 0.0" rpy="0.0 0.0 0.0"/>
-            <geometry>
-                <mesh filename="package://arm_description/meshes/collision/arm_link_2.stl" scale="0.001 0.001 0.001"/>
-            </geometry>
-        </collision>
-    </link>
-    <joint name="arm_joint_2" type="revolute">
-        <parent link="arm_link_2"/>
-        <child link="arm_link_3"/>
-        <origin xyz="0.0 0.0 0.04" rpy="0.0 0.0 0.0"/>
-        <axis xyz="0 1 0"/>
-        <dynamics damping="0"/>
-        <dynamics friction="0"/>
-        <limit effort="87" velocity="5.6548668" lower="-2.6179939" upper="2.6179939" />
-    </joint>
-    <link name="arm_link_3">
-        <inertial>
-            <origin xyz="0.0 0.0 0.0" rpy="0.0 0.0 0.0"/>
-            <mass value="0.1"/>
-            <inertia ixx="0.001" ixy="0.001" ixz="0.001" iyy="0.001" iyz="0.001" izz="0.001"/>
-        </inertial>
-        <visual>
-            <origin xyz="0.0 0.0 0.0" rpy="0.0 0.0 ${pi/2.0}"/>
-            <geometry>
-                <mesh filename="package://arm_description/meshes/visual/arm_link_3.stl" scale="0.001 0.001 0.001"/>
-            </geometry>
-            <material name="Grey">
-                <color rgba="0.2 0.2 0.2 1"/>
-            </material>
-        </visual>
-        <collision>
-            <origin xyz="0.0 0.0 0.0" rpy="0.0 0.0 ${pi/2}"/>
-            <geometry>
-                <mesh filename="package://arm_description/meshes/collision/arm_link_3.stl" scale="0.001 0.001 0.001"/>
-            </geometry>
-        </collision>
-    </link>
-    <joint name="arm_joint_3" type="revolute">
-        <parent link="arm_link_3"/>
-        <child link="arm_link_4"/>
-        <origin xyz="-0.3683 0.014 0.073" rpy="0.0 ${pi} 0.0"/>
-        <axis xyz="0 1 0"/>
-        <dynamics damping="0"/>
-        <dynamics friction="0"/>
-        <limit effort="87" velocity="5.6548668" lower="-2.6179939" upper="2.6179939" />
-    </joint>
-    <link name="arm_link_4">
-        <inertial>
-            <origin xyz="0.0 0.0 0.0" rpy="0.0 0.0 0.0"/>
-            <mass value="0.1"/>
-            <inertia ixx="0.001" ixy="0.001" ixz="0.001" iyy="0.001" iyz="0.001" izz="0.001"/>
-        </inertial>
-        <visual>
-            <origin xyz="0.0 0.0 0.0" rpy="0.0 0.0 ${pi/2.0}"/>
-            <geometry>
-                <mesh filename="package://arm_description/meshes/visual/arm_link_4.stl" scale="0.001 0.001 0.001"/>
-            </geometry>
-            <material name="Grey">
-                <color rgba="0.2 0.2 0.2 1"/>
-            </material>
-        </visual>
-        <collision>
-            <origin xyz="0.0 0.0 0.0" rpy="0.0 0.0 ${pi/2}"/>
-            <geometry>
-                <mesh filename="package://arm_description/meshes/collision/arm_link_4.stl" scale="0.001 0.001 0.001"/>
-            </geometry>
-        </collision>
-    </link>
-    <joint name="arm_joint_4" type="revolute">
-        <parent link="arm_link_4"/>
-        <child link="arm_link_5"/>
-        <origin xyz="-0.202 0.0 0.0" rpy="0.0 ${pi} 0.0"/>
-        <axis xyz="1 0 0"/>
-        <dynamics damping="0"/>
-        <dynamics friction="0"/>
-        <limit effort="87" velocity="5.6548668" lower="-2.6179939" upper="2.6179939" />
-    </joint>
-    <link name="arm_link_5">
-        <inertial>
-            <origin xyz="0.0 0.0 0.0" rpy="0.0 0.0 0.0"/>
-            <mass value="0.1"/>
-            <inertia ixx="0.001" ixy="0.001" ixz="0.001" iyy="0.001" iyz="0.001" izz="0.001"/>
-        </inertial>
-        <visual>
-            <origin xyz="0.0 0.0 0.0" rpy="0.0 0.0 0.0"/>
-            <geometry>
-                <mesh filename="package://arm_description/meshes/visual/arm_link_5.stl" scale="0.001 0.001 0.001"/>
-            </geometry>
-            <material name="Grey">
-                <color rgba="0.2 0.2 0.2 1"/>
-            </material>
-        </visual>
-        <collision>
-            <origin xyz="0.0 0.0 0.0" rpy="0.0 0.0 0.0"/>
-            <geometry>
-                <mesh filename="package://arm_description/meshes/collision/arm_link_5.stl" scale="0.001 0.001 0.001"/>
-            </geometry>
-        </collision>
-    </link>
-    <joint name="arm_joint_5" type="revolute">
-        <parent link="arm_link_5"/>
-        <child link="arm_link_6"/>
-        <origin xyz="0.17875 0.0 0.0" rpy="0.0 0.0 0.0"/>
-        <axis xyz="0 1 0"/>
-        <dynamics damping="0"/>
-        <dynamics friction="0"/>
-        <limit effort="87" velocity="5.6548668" lower="-2.6179939" upper="2.6179939" />
-    </joint>
-    <link name="arm_link_6">
-        <inertial>
-            <origin xyz="0.0 0.0 0.0" rpy="0.0 0.0 0.0"/>
-            <mass value="0.1"/>
-            <inertia ixx="0.001" ixy="0.001" ixz="0.001" iyy="0.001" iyz="0.001" izz="0.001"/>
-        </inertial>
-        <visual>
-            <origin xyz="0.0 0.0 0.0" rpy="0.0 0.0 0.0"/>
-            <geometry>
-                <mesh filename="package://arm_description/meshes/visual/arm_link_6.stl" scale="0.001 0.001 0.001"/>
-            </geometry>
-            <material name="Grey">
-                <color rgba="0.2 0.2 0.2 1"/>
-            </material>
-        </visual>
-        <collision>
-            <origin xyz="0.0 0.0 0.0" rpy="0.0 0.0 0.0"/>
-            <geometry>
-                <mesh filename="package://arm_description/meshes/collision/arm_link_6.stl" scale="0.001 0.001 0.001"/>
-            </geometry>
-        </collision>
-    </link>
-</xacro:macro>
+    <!-- All meshes are scaled by 0.001 in all dimensions because I exported in mm, ROS uses m-->
+    <xacro:macro name="hexapod_arm" params="parent xyz rpy">
+        <joint name="arm_attachment" type="fixed">
+            <parent link="${parent}"/>
+            <child link="arm_link_1"/>
+            <origin xyz="${xyz}" rpy="${rpy}"/>
+        </joint>
+        <link name="arm_link_1">
+            <inertial>
+                <origin xyz="0.0 0.0 0.0" rpy="0.0 0.0 0.0"/>
+                <mass value="0.1"/>
+                <inertia ixx="0.001" ixy="0.001" ixz="0.001" iyy="0.001" iyz="0.001" izz="0.001"/>
+            </inertial>
+            <visual>
+                <origin xyz="0 0 0.0" rpy="0.0 0.0 0.0"/>
+                <geometry>
+                    <mesh filename="package://arm_description/meshes/visual/arm_link_1.stl" scale="0.001 0.001 0.001"/>
+                </geometry>
+                <material name="Grey">
+                    <color rgba="0.2 0.2 0.2 1"/>
+                </material>
+            </visual>
+            <collision>
+                <origin xyz="0.0 0.0 0.0" rpy="0.0 0.0 0.0"/>
+                <geometry>
+                    <mesh filename="package://arm_description/meshes/collision/arm_link_1.stl" scale="0.001 0.001 0.001"/>
+                </geometry>
+            </collision>
+        </link>
+        <joint name="arm_joint_1" type="revolute">
+            <parent link="arm_link_1"/>
+            <child link="arm_link_2"/>
+            <origin xyz="0.0 0.0 0.194" rpy="0.0 0.0 ${5*pi/4.0}"/>
+            <axis xyz="0 0 1"/>
+            <dynamics damping="0"/>
+            <dynamics friction="0"/>
+            <limit effort="87" velocity="5.6548668" lower="-2.6179939" upper="2.6179939" />
+        </joint>
+        <link name="arm_link_2">
+            <inertial>
+                <origin xyz="0.0 0.0 0.0" rpy="0.0 0.0 0.0"/>
+                <mass value="0.1"/>
+                <inertia ixx="0.001" ixy="0.001" ixz="0.001" iyy="0.001" iyz="0.001" izz="0.001"/>
+            </inertial>
+            <visual>
+                <origin xyz="0.0 0.0 0.0" rpy="0.0 0.0 0.0"/>
+                <geometry>
+                    <mesh filename="package://arm_description/meshes/visual/arm_link_2.stl" scale="0.001 0.001 0.001"/>
+                </geometry>
+                <material name="Grey">
+                    <color rgba="0.2 0.2 0.2 1"/>
+                </material>
+            </visual>
+            <collision>
+                <origin xyz="0.0 0.0 0.0" rpy="0.0 0.0 0.0"/>
+                <geometry>
+                    <mesh filename="package://arm_description/meshes/collision/arm_link_2.stl" scale="0.001 0.001 0.001"/>
+                </geometry>
+            </collision>
+        </link>
+        <joint name="arm_joint_2" type="revolute">
+            <parent link="arm_link_2"/>
+            <child link="arm_link_3"/>
+            <origin xyz="0.0 0.0 0.04" rpy="0.0 0.0 0.0"/>
+            <axis xyz="0 1 0"/>
+            <dynamics damping="0"/>
+            <dynamics friction="0"/>
+            <limit effort="87" velocity="5.6548668" lower="-2.6179939" upper="2.6179939" />
+        </joint>
+        <link name="arm_link_3">
+            <inertial>
+                <origin xyz="0.0 0.0 0.0" rpy="0.0 0.0 0.0"/>
+                <mass value="0.1"/>
+                <inertia ixx="0.001" ixy="0.001" ixz="0.001" iyy="0.001" iyz="0.001" izz="0.001"/>
+            </inertial>
+            <visual>
+                <origin xyz="0.0 0.0 0.0" rpy="0.0 0.0 ${pi/2.0}"/>
+                <geometry>
+                    <mesh filename="package://arm_description/meshes/visual/arm_link_3.stl" scale="0.001 0.001 0.001"/>
+                </geometry>
+                <material name="Grey">
+                    <color rgba="0.2 0.2 0.2 1"/>
+                </material>
+            </visual>
+            <collision>
+                <origin xyz="0.0 0.0 0.0" rpy="0.0 0.0 ${pi/2}"/>
+                <geometry>
+                    <mesh filename="package://arm_description/meshes/collision/arm_link_3.stl" scale="0.001 0.001 0.001"/>
+                </geometry>
+            </collision>
+        </link>
+        <joint name="arm_joint_3" type="revolute">
+            <parent link="arm_link_3"/>
+            <child link="arm_link_4"/>
+            <origin xyz="-0.3683 0.014 0.073" rpy="0.0 ${pi} 0.0"/>
+            <axis xyz="0 1 0"/>
+            <dynamics damping="0"/>
+            <dynamics friction="0"/>
+            <limit effort="87" velocity="5.6548668" lower="-2.6179939" upper="2.6179939" />
+        </joint>
+        <link name="arm_link_4">
+            <inertial>
+                <origin xyz="0.0 0.0 0.0" rpy="0.0 0.0 0.0"/>
+                <mass value="0.1"/>
+                <inertia ixx="0.001" ixy="0.001" ixz="0.001" iyy="0.001" iyz="0.001" izz="0.001"/>
+            </inertial>
+            <visual>
+                <origin xyz="0.0 0.0 0.0" rpy="0.0 0.0 ${pi/2.0}"/>
+                <geometry>
+                    <mesh filename="package://arm_description/meshes/visual/arm_link_4.stl" scale="0.001 0.001 0.001"/>
+                </geometry>
+                <material name="Grey">
+                    <color rgba="0.2 0.2 0.2 1"/>
+                </material>
+            </visual>
+            <collision>
+                <origin xyz="0.0 0.0 0.0" rpy="0.0 0.0 ${pi/2}"/>
+                <geometry>
+                    <mesh filename="package://arm_description/meshes/collision/arm_link_4.stl" scale="0.001 0.001 0.001"/>
+                </geometry>
+            </collision>
+        </link>
+        <joint name="arm_joint_4" type="revolute">
+            <parent link="arm_link_4"/>
+            <child link="arm_link_5"/>
+            <origin xyz="-0.202 0.0 0.0" rpy="0.0 ${pi} 0.0"/>
+            <axis xyz="1 0 0"/>
+            <dynamics damping="0"/>
+            <dynamics friction="0"/>
+            <limit effort="87" velocity="5.6548668" lower="-2.6179939" upper="2.6179939" />
+        </joint>
+        <link name="arm_link_5">
+            <inertial>
+                <origin xyz="0.0 0.0 0.0" rpy="0.0 0.0 0.0"/>
+                <mass value="0.1"/>
+                <inertia ixx="0.001" ixy="0.001" ixz="0.001" iyy="0.001" iyz="0.001" izz="0.001"/>
+            </inertial>
+            <visual>
+                <origin xyz="0.0 0.0 0.0" rpy="0.0 0.0 0.0"/>
+                <geometry>
+                    <mesh filename="package://arm_description/meshes/visual/arm_link_5.stl" scale="0.001 0.001 0.001"/>
+                </geometry>
+                <material name="Grey">
+                    <color rgba="0.2 0.2 0.2 1"/>
+                </material>
+            </visual>
+            <collision>
+                <origin xyz="0.0 0.0 0.0" rpy="0.0 0.0 0.0"/>
+                <geometry>
+                    <mesh filename="package://arm_description/meshes/collision/arm_link_5.stl" scale="0.001 0.001 0.001"/>
+                </geometry>
+            </collision>
+        </link>
+        <joint name="arm_joint_5" type="revolute">
+            <parent link="arm_link_5"/>
+            <child link="arm_link_6"/>
+            <origin xyz="0.17875 0.0 0.0" rpy="0.0 0.0 0.0"/>
+            <axis xyz="0 1 0"/>
+            <dynamics damping="0"/>
+            <dynamics friction="0"/>
+            <limit effort="87" velocity="5.6548668" lower="-2.6179939" upper="2.6179939" />
+        </joint>
+        <link name="arm_link_6">
+            <inertial>
+                <origin xyz="0.0 0.0 0.0" rpy="0.0 0.0 0.0"/>
+                <mass value="0.1"/>
+                <inertia ixx="0.001" ixy="0.001" ixz="0.001" iyy="0.001" iyz="0.001" izz="0.001"/>
+            </inertial>
+            <visual>
+                <origin xyz="0.0 0.0 0.0" rpy="0.0 0.0 0.0"/>
+                <geometry>
+                    <mesh filename="package://arm_description/meshes/visual/arm_link_6.stl" scale="0.001 0.001 0.001"/>
+                </geometry>
+                <material name="Grey">
+                    <color rgba="0.2 0.2 0.2 1"/>
+                </material>
+            </visual>
+            <collision>
+                <origin xyz="0.0 0.0 0.0" rpy="0.0 0.0 0.0"/>
+                <geometry>
+                    <mesh filename="package://arm_description/meshes/collision/arm_link_6.stl" scale="0.001 0.001 0.001"/>
+                </geometry>
+            </collision>
+        </link>
+    </xacro:macro>
 </robot>

File: arm_description/urdf/arm.xacro (robot description, xacro)
@@ -3,5 +3,5 @@
     <xacro:include filename="$(find arm_description)/urdf/arm.urdf.xacro" />
     <link name="base_link"/>
-    <xacro:hexapod_arm parent="base_link"/>
+    <xacro:hexapod_arm parent="base_link" xyz="0 0 0" rpy="0 0 0"/>
     <!-- Fix to floor for gazebo testing -->
     <link name="world"/>

Commit message: Fixed gazebo glitch with hexapod base, changed inertia matrices. Restructured URDF files for hexapod base

File: arm_description/urdf/arm.urdf.xacro (robot description, xacro)
@@ -185,4 +185,5 @@
             </collision>
         </link>
+        <xacro:include filename="$(find arm_description)/urdf/arm.transmission.xacro"/>
     </xacro:macro>
 </robot>

File: hexapod_description/urdf/hexapod.urdf.xacro (robot description, xacro)
@@ -10,6 +10,6 @@
             <inertial>
                 <origin xyz="0.0 0.0 0.0" rpy="0.0 0.0 0.0"/>
-                <mass value="0.1"/>
-                <inertia ixx="0.001" ixy="0.001" ixz="0.001" iyy="0.001" iyz="0.001" izz="0.001"/>
+                <mass value="1"/>
+                <inertia ixx="0.001" ixy="0.0" ixz="0.0" iyy="0.001" iyz="0.0" izz="0.001"/>
             </inertial>
             <visual>
@@ -43,10 +43,11 @@
             <axis xyz="0 0 1"/>
             <limit effort="87" velocity="5.6548668" lower="-2.6179939" upper="2.6179939" />
+            <dynamics damping="1.0"/>
         </joint>
         <link name="coxa_link_${suffix}">
             <inertial>
                 <origin xyz="0.0 0.0 0.0" rpy="0.0 0.0 0.0"/>
-                <mass value="0.1"/>
-                <inertia ixx="0.001" ixy="0.001" ixz="0.001" iyy="0.001" iyz="0.001" izz="0.001"/>
+                <mass value="1"/>
+                <inertia ixx="0.001" ixy="0.0" ixz="0.0" iyy="0.001" iyz="0.0" izz="0.001"/>
             </inertial>
             <visual>
@@ -72,10 +73,11 @@
             <axis xyz="0 1 0"/>
             <limit effort="87" velocity="5.6548668" lower="-2.6179939" upper="2.6179939" />
+            <dynamics damping="1.0"/>
         </joint>
         <link name="thigh_link_${suffix}">
             <inertial>
                 <origin xyz="0.0 0.0 0.0" rpy="0.0 0.0 0.0"/>
-                <mass value="0.1"/>
-                <inertia ixx="0.001" ixy="0.001" ixz="0.001" iyy="0.001" iyz="0.001" izz="0.001"/>
+                <mass value="1"/>
+                <inertia ixx="0.001" ixy="0.0" ixz="0.0" iyy="0.001" iyz="0.0" izz="0.001"/>
             </inertial>
             <visual>
@@ -101,10 +103,11 @@
             <axis xyz="0 1 0"/>
             <limit effort="87" velocity="5.6548668" lower="-2.6179939" upper="2.6179939" />
+            <dynamics damping="1.0"/>
         </joint>
         <link name="tibia_link_${suffix}">
             <inertial>
                 <origin xyz="0.0 0.0 0.0" rpy="0.0 0.0 0.0"/>
-                <mass value="0.1"/>
-                <inertia ixx="0.001" ixy="0.001" ixz="0.001" iyy="0.001" iyz="0.001" izz="0.001"/>
+                <mass value="1"/>
+                <inertia ixx="0.001" ixy="0.0" ixz="0.0" iyy="0.001" iyz="0.0" izz="0.001"/>
             </inertial>
             <visual>
@@ -124,4 +127,6 @@
             </collision>
         </link>
+        <xacro:include filename="$(find hexapod_description)/urdf/hexapod.transmission.xacro"/>
+        <xacro:leg_joint_transmission suffix="${suffix}"/>
     </xacro:macro>
 </robot>

File: hexapod_description/urdf/hexapod.xacro (robot description, xacro)
@@ -4,3 +4,5 @@
     <link name="base_link"/>
     <xacro:hexapod_base parent="base_link"/>
+    <xacro:include filename="$(find hexapod_description)/urdf/hexapod.gazebo.xacro"/>
+    <xacro:hexapod_gazebo/>
 </robot>

File: hexapod_description/urdf/hexapod_arm.xacro (robot description, xacro)
@@ -1,8 +1,10 @@
 <?xml version="1.0" ?>
 <robot name="hexapod_with_arm" xmlns:xacro="http://www.ros.org/wiki/xacro">
-    <xacro:include filename="$(find hexapod_description)/urdf/hexapod.urdf.xacro" />
-    <xacro:include filename="$(find arm_description)/urdf/arm.urdf.xacro" />
+    <xacro:include filename="$(find hexapod_description)/urdf/hexapod.urdf.xacro"/>
+    <xacro:include filename="$(find arm_description)/urdf/arm.urdf.xacro"/>
     <link name="base_link"/>
     <xacro:hexapod_base parent="base_link"/>
     <xacro:hexapod_arm parent="body_link" xyz="0.1809 0 -0.0489" rpy="0 0 ${3*pi/4.0}"/>
+    <xacro:include filename="$(find hexapod_description)/urdf/hexapod.gazebo.xacro"/>
+    <xacro:hexapod_gazebo/>
 </robot>
