Commit message: New MoveIt config generated for arm. Tested with Gazebo

File: arm_description/urdf/arm.urdf.xacro (robot description, xacro)
@@ -12,5 +12,5 @@
                 <origin xyz="0.0 0.0 0.0" rpy="0.0 0.0 0.0"/>
                 <mass value="0.1"/>
-                <inertia ixx="0.001" ixy="0.001" ixz="0.001" iyy="0.001" iyz="0.001" izz="0.001"/>
+                <inertia ixx="0.001" ixy="0.0" ixz="0.0" iyy="0.001" iyz="0.0" izz="0.001"/>
             </inertial>
             <visual>
@@ -43,5 +43,5 @@
                 <origin xyz="0.0 0.0 0.0" rpy="0.0 0.0 0.0"/>
                 <mass value="0.1"/>
-                <inertia ixx="0.001" ixy="0.001" ixz="0.001" iyy="0.001" iyz="0.001" izz="0.001"/>
+                <inertia ixx="0.001" ixy="0.0" ixz="0.0" iyy="0.001" iyz="0.0" izz="0.001"/>
             </inertial>
             <visual>
@@ -74,5 +74,5 @@
                 <origin xyz="0.0 0.0 0.0" rpy="0.0 0.0 0.0"/>
                 <mass value="0.1"/>
-                <inertia ixx="0.001" ixy="0.001" ixz="0.001" iyy="0.001" iyz="0.001" izz="0.001"/>
+                <inertia ixx="0.001" ixy="0.0" ixz="0.0" iyy="0.001" iyz="0.0" izz="0.001"/>
             </inertial>
             <visual>
@@ -105,5 +105,5 @@
                 <origin xyz="0.0 0.0 0.0" rpy="0.0 0.0 0.0"/>
                 <mass value="0.1"/>
-                <inertia ixx="0.001" ixy="0.001" ixz="0.001" iyy="0.001" iyz="0.001" izz="0.001"/>
+                <inertia ixx="0.001" ixy="0.0" ixz="0.0" iyy="0.001" iyz="0.0" izz="0.001"/>
             </inertial>
             <visual>
@@ -136,5 +136,5 @@
                 <origin xyz="0.0 0.0 0.0" rpy="0.0 0.0 0.0"/>
                 <mass value="0.1"/>
-                <inertia ixx="0.001" ixy="0.001" ixz="0.001" iyy="0.001" iyz="0.001" izz="0.001"/>
+                <inertia ixx="0.001" ixy="0.0" ixz="0.0" iyy="0.001" iyz="0.0" izz="0.001"/>
             </inertial>
             <visual>
@@ -167,5 +167,5 @@
                 <origin xyz="0.0 0.0 0.0" rpy="0.0 0.0 0.0"/>
                 <mass value="0.1"/>
-                <inertia ixx="0.001" ixy="0.001" ixz="0.001" iyy="0.001" iyz="0.001" izz="0.001"/>
+                <inertia ixx="0.001" ixy="0.0" ixz="0.0" iyy="0.001" iyz="0.0" izz="0.001"/>
             </inertial>
             <visual>

File: hexapod_description/urdf/hexapod.gazebo.xacro (robot description, xacro)
@@ -14,9 +14,4 @@
         <xacro:leg_gazebo suffix="rm"/>
         <xacro:leg_gazebo suffix="rr"/>
-        <gazebo>
-            <plugin name="ros_control" filename="libgazebo_ros_control.so">
-              <robotNamespace></robotNamespace>
-            </plugin>
-        </gazebo>
     </xacro:macro>
     <xacro:macro name="leg_gazebo" params="suffix">

File: hexapod_description/urdf/hexapod_arm.xacro (robot description, xacro)
@@ -6,5 +6,13 @@
     <xacro:hexapod_base parent="base_link"/>
     <xacro:hexapod_arm parent="body_link" xyz="0.1809 0 -0.0489" rpy="0 0 ${3*pi/4.0}"/>
+    <!--Include Gazebo components-->
     <xacro:include filename="$(find hexapod_description)/urdf/hexapod.gazebo.xacro"/>
     <xacro:hexapod_gazebo/>
+    <xacro:include filename="$(find arm_description)/urdf/arm.gazebo.xacro"/>
+    <xacro:arm_gazebo/>
+    <gazebo>
+        <plugin name="ros_control" filename="libgazebo_ros_control.so">
+          <robotNamespace></robotNamespace>
+        </plugin>
+    </gazebo>
 </robot>

Commit message: Simple walking script working, adapted from phantomx_gazebo. Joint limits updated in URDF

File: arm_description/urdf/arm.urdf.xacro (robot description, xacro)
@@ -37,5 +37,5 @@
             <dynamics damping="0"/>
             <dynamics friction="0"/>
-            <limit effort="87" velocity="5.6548668" lower="-2.6179939" upper="2.6179939" />
+            <limit effort="87" velocity="5.6548668" lower="-3.14" upper="3.14" />
         </joint>
         <link name="arm_link_2">
@@ -68,5 +68,5 @@
             <dynamics damping="0"/>
             <dynamics friction="0"/>
-            <limit effort="87" velocity="5.6548668" lower="-2.6179939" upper="2.6179939" />
+            <limit effort="87" velocity="5.6548668" lower="0" upper="3.14" />
         </joint>
         <link name="arm_link_3">
@@ -99,5 +99,5 @@
             <dynamics damping="0"/>
             <dynamics friction="0"/>
-            <limit effort="87" velocity="5.6548668" lower="-2.6179939" upper="2.6179939" />
+            <limit effort="87" velocity="5.6548668" lower="-3.14" upper="0" />
         </joint>
         <link name="arm_link_4">
@@ -130,5 +130,5 @@
             <dynamics damping="0"/>
             <dynamics friction="0"/>
-            <limit effort="87" velocity="5.6548668" lower="-2.6179939" upper="2.6179939" />
+            <limit effort="87" velocity="5.6548668" lower="-3.14" upper="3.14" />
         </joint>
         <link name="arm_link_5">
@@ -161,5 +161,5 @@
             <dynamics damping="0"/>
             <dynamics friction="0"/>
-            <limit effort="87" velocity="5.6548668" lower="-2.6179939" upper="2.6179939" />
+            <limit effort="87" velocity="5.6548668" lower="-1.57" upper="1.57" />
         </joint>
         <link name="arm_link_6">

File: hexapod_description/urdf/hexapod.urdf.xacro (robot description, xacro)
@@ -96,5 +96,13 @@
             <origin xyz="${xyz}" rpy="${rpy}"/>
             <axis xyz="0 0 1"/>
-            <limit effort="87" velocity="5.6548668" lower="-2.6179939" upper="2.6179939" />
+            <xacro:if value="${suffix == 'lm' or suffix == 'rm'}">
+                <limit effort="87" velocity="5.6548668" lower="-0.75" upper="0.75"/>
+            </xacro:if>
+            <xacro:if value="${suffix == 'lf' or suffix == 'rr'}">
+                <limit effort="87" velocity="5.6548668" lower="-0.5" upper="1.5"/>
+            </xacro:if>
+            <xacro:if value="${suffix == 'rf' or suffix == 'lr'}">
+                <limit effort="87" velocity="5.6548668" lower="-1.5" upper="0.5"/>
+            </xacro:if>
             <dynamics damping="1.0"/>
         </joint>
@@ -126,5 +134,5 @@
             <origin xyz="0.1 0.0 0.0" rpy="0.0 0.0 0.0"/>
             <axis xyz="0 1 0"/>
-            <limit effort="87" velocity="5.6548668" lower="-2.6179939" upper="2.6179939" />
+            <limit effort="87" velocity="5.6548668" lower="-0.68" upper="2.62" />
             <dynamics damping="1.0"/>
         </joint>
@@ -154,7 +162,7 @@
             <parent link="thigh_link_${suffix}"/>
             <child link="tibia_link_${suffix}"/>
-            <origin xyz="0.1199 0.0 0.07597" rpy="0.0 0.0 0.0"/>
-            <axis xyz="0 1 0"/>
-            <limit effort="87" velocity="5.6548668" lower="-2.6179939" upper="2.6179939" />
+            <origin xyz="0.1199 -0.005 0.07597" rpy="0.0 0.0 0.0"/>
+            <axis xyz="0 -1 0"/>
+            <limit effort="87" velocity="5.6548668" lower="-0.42" upper="2.44" />
             <dynamics damping="1.0"/>
         </joint>

File: hexapod_description/urdf/hexapod.xacro (robot description, xacro)
@@ -5,4 +5,8 @@
     <xacro:hexapod_base parent="base_link"/>
     <xacro:include filename="$(find hexapod_description)/urdf/hexapod.gazebo.xacro"/>
-    <xacro:hexapod_gazebo/>
+    <gazebo>
+        <plugin name="ros_control" filename="libgazebo_ros_control.so">
+          <robotNamespace></robotNamespace>
+        </plugin>
+    </gazebo>
 </robot>
