Commit message: Implemented control for hexapod

File: hexapod_description/urdf/hexapod.gazebo.xacro (robot description, xacro)
@@ -88,5 +88,5 @@
             <maxVel>0</maxVel>
         </gazebo>
-        <gazebo reference="thigh_link_${suffix}">
+        <gazebo reference="femur_link_${suffix}">
             <material>Gazebo/Grey</material>
             <mu1>0.2</mu1>

File: hexapod_description/urdf/hexapod.transmission.xacro (robot description, xacro)
@@ -12,10 +12,10 @@
             </actuator>
         </transmission>
-        <transmission name="thigh_joint_${suffix}_transmission">
+        <transmission name="femur_joint_${suffix}_transmission">
             <type>transmission_interface/SimpleTransmission</type>
-            <joint name="thigh_joint_${suffix}">
+            <joint name="femur_joint_${suffix}">
                 <hardwareInterface>hardware_interface/EffortJointInterface</hardwareInterface>
             </joint>
-            <actuator name="thigh_joint_${suffix}_motor">
+            <actuator name="femur_joint_${suffix}_motor">
                 <hardwareInterface>hardware_interface/EffortJointInterface</hardwareInterface>
                 <mechanicalReduction>1</mechanicalReduction>

File: hexapod_description/urdf/hexapod.urdf.xacro (robot description, xacro)
@@ -121,7 +121,7 @@
             </collision>
         </link>
-        <joint name="thigh_joint_${suffix}" type="revolute">
+        <joint name="femur_joint_${suffix}" type="revolute">
             <parent link="coxa_link_${suffix}"/>
-            <child link="thigh_link_${suffix}"/>
+            <child link="femur_link_${suffix}"/>
             <origin xyz="0.1 0.0 0.0" rpy="0.0 0.0 0.0"/>
             <axis xyz="0 1 0"/>
@@ -129,5 +129,5 @@
             <dynamics damping="1.0"/>
         </joint>
-        <link name="thigh_link_${suffix}">
+        <link name="femur_link_${suffix}">
             <inertial>
                 <origin xyz="0.0 0.0 0.0" rpy="0.0 0.0 0.0"/>
@@ -152,5 +152,5 @@
         </link>
         <joint name="tibia_joint_${suffix}" type="revolute">
-            <parent link="thigh_link_${suffix}"/>
+            <parent link="femur_link_${suffix}"/>
             <child link="tibia_link_${suffix}"/>
             <origin xyz="0.1199 0.0 0.07597" rpy="0.0 0.0 0.0"/>
